File: DSI_CSI.kicad_sch (KiCad schematic)
At the start: 1 part, among them J802 Conn_01x22_Female

Commit message: power symbols
Connections:
- net 3V3 renamed +3V3_PI
Changed lines of the file:
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@@
 	(wire
 		(pts
-			(xy 19.05 27.94) (xy 29.21 27.94)
-		)
-		(stroke
-			(width 0)
-			(type default)
-		)
-	)
-	(wire
-		(pts
-			(xy 106.68 87.63) (xy 88.9 87.63)
+			(xy 106.68 87.63) (xy 82.55 87.63)
 		)
 		(stroke
@@
 		)
 	)
-	(label "_3V3"
-		(at 29.21 27.94 180)
-		(fields_autoplaced yes)
-		(effects
-			(font
-				(size 1.27 1.27)
-			)
-			(justify right bottom)
-		)
-	)
 	(label "DPHY0_C.D0_P"
 		(at 90.17 39.37 0)
@@
 		)
 	)
-	(label "_3V3"
-		(at 88.9 87.63 0)
-		(fields_autoplaced yes)
-		(effects
-			(font
-				(size 1.27 1.27)
-			)
-			(justify left bottom)
-		)
-	)
 	(label "DPHY0_C.D3_P"
 		(at 90.17 69.85 0)
@@
 			)
 			(justify left bottom)
-		)
-	)
-	(hierarchical_label "3V3"
-		(shape input)
-		(at 19.05 27.94 180)
-		(fields_autoplaced yes)
-		(effects
-			(font
-				(size 1.27 1.27)
-			)
-			(justify right)
 		)
 	)
@@
 	)
 	(hierarchical_label "CAM_GPIO1"
-		(shape input)
+		(shape output)
 		(at 99.06 77.47 180)
 		(fields_autoplaced yes)
@@
 	)
 	(hierarchical_label "CAM_GPIO0"
-		(shape input)
+		(shape output)
 		(at 99.06 74.93 180)
 		(fields_autoplaced yes)
@@
 	)
 	(hierarchical_label "DPHY0_C{DPHY}"
-		(shape input)
+		(shape bidirectional)
 		(at 82.55 31.75 180)
 		(fields_autoplaced yes)
@@
 		)
 	)
+	(symbol
+		(lib_id "power:+3V3")
+		(at 82.55 87.63 0)
+		(unit 1)
+		(exclude_from_sim no)
+		(in_bom yes)
+		(on_board yes)
+		(dnp no)
+		(property "Reference" "#PWR0801"
+			(at 82.55 91.44 0)
+			(effects
+				(font
+					(size 1.27 1.27)
+				)
+				(hide yes)
+			)
+		)
+		(property "Value" "+3V3_PI"
+			(at 78.994 83.058 0)
+			(effects
+				(font
+					(size 1.27 1.27)
+				)
+				(justify left)
+			)
+		)
+		(property "Footprint" ""
+			(at 82.55 87.63 0)
+			(effects
+				(font
+					(size 1.27 1.27)
+				)
+				(hide yes)
+			)
+		)
+		(property "Datasheet" ""
+			(at 82.55 87.63 0)
+			(effects
+				(font
+					(size 1.27 1.27)
+				)
+				(hide yes)
+			)
+		)
+		(property "Description" "Power symbol creates a global label with name \"+3V3\""
+			(at 82.55 87.63 0)
+			(effects
+				(font
+					(size 1.27 1.27)
+				)
+				(hide yes)
+			)
+		)
+		(pin "1"
+		)
+		(instances
+			(project "CM5_MINIMA_2"
+				(path "/b33e81d6-18a9-4b9d-a239-76a7c253462f/dfe055fd-896e-497d-b242-c071b2f18dd1"
+					(reference "#PWR0801")
+					(unit 1)
+				)
+			)
+		)
+	)
