File: PCIe-M2.kicad_sch (KiCad schematic)
At the start: 21 parts, among them J701 Bus_M.2_Socket_M, M701 M.2 Solder Nut, M705 M.2 Screw, U702 AP3441SHE-7B, U703 ASEK-32.768KHZ-L-R-T

Commit message: power symbols
Connections:
- net GND: no longer J701.M2 (GND2242), J701.M3 (GND2260), J701.M4 (GND2280)
- net +5v renamed +5V
- net M2_3v3 renamed M2_3V3
- net PCIE_C._PWR_EN renamed PCIE_C.PWR_EN
