File: PCIe-M2.kicad_sch (KiCad schematic)
At the start: 21 parts, among them J701 Bus_M.2_Socket_M, M701 M.2 Solder Nut, M705 M.2 Screw, U702 AP3441SHE-7B, U703 ASEK-32.768KHZ-L-R-T

Commit message: swap TX RX M2
Connections:
- net RX: now also J701.22 (NC); no longer J701.20 (NC)
- net TX: now also J701.20 (NC); no longer J701.22 (NC)
Changed lines of the file:
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@@
 	(hierarchical_label "TX"
 		(shape input)
-		(at 185.42 74.93 0)
+		(at 185.42 77.47 0)
 		(fields_autoplaced yes)
 		(effects
@@
 	(hierarchical_label "RX"
 		(shape input)
-		(at 185.42 77.47 0)
+		(at 185.42 74.93 0)
 		(fields_autoplaced yes)
 		(effects

Commit message: prod
Parts:
- R707: value 1k -> 2k2
Changed lines of the file:
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@@
 			)
 		)
-		(property "Value" "1k"
+		(property "Value" "2k2"
 			(at 197.358 83.693 0)
 			(effects

Commit message: jlc bom polishing
Parts:
- M701: footprint (none) -> MountingHole:MountingHole_3.78mm_M2_Pad_TopOnly
- R704: value 100K 1% -> 100k; Field4 Farnell -> (none); Field6 MCR01MZPF1003 -> (none); Field7 Rohm -> (none); Part Description Resistor 100K M1005 1% 63mW -> (none)
- R705: value 10K 1% -> 10k; Field4 Farnell -> (none); Field6 MCR01MZPF1002 -> (none); Field7 Rohm -> (none); Part Description Resistor 10K M1005 1% 63mW -> (none)
- R706: value 2.2K 1% -> 2k2; Field4 Farnell -> (none); Part Description Resistor 2.2K M1005 1% 63mW -> (none)
Changed lines of the file:
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@@
 			)
 		)
-		(property "Value" "10K 1%"
+		(property "Value" "10k"
 			(at 114.808 172.593 0)
 			(effects
@@
 			)
 		)
-		(property "Datasheet" "https://fscdn.rohm.com/en/products/databook/datasheet/passive/resistor/chip_resistor/mcr-e.pdf"
+		(property "Datasheet" ""
 			(at 113.03 171.45 0)
 			(effects
@@
 		)
 		(property "Description" ""
-			(at 113.03 171.45 0)
-			(effects
-				(font
-					(size 1.27 1.27)
-				)
-				(hide yes)
-			)
-		)
-		(property "Field4" "Farnell"
-			(at 113.03 171.45 0)
-			(effects
-				(font
-					(size 1.27 1.27)
-				)
-				(hide yes)
-			)
-		)
-		(property "Field5" ""
-			(at 113.03 171.45 0)
-			(effects
-				(font
-					(size 1.27 1.27)
-				)
-				(hide yes)
-			)
-		)
-		(property "Field7" "Rohm"
-			(at 113.03 171.45 0)
-			(effects
-				(font
-					(size 1.27 1.27)
-				)
-				(hide yes)
-			)
-		)
-		(property "Field6" "MCR01MZPF1002"
-			(at 113.03 171.45 0)
-			(effects
-				(font
-					(size 1.27 1.27)
-				)
-				(hide yes)
-			)
-		)
-		(property "Part Description" "Resistor 10K M1005 1% 63mW"
 			(at 113.03 171.45 0)
 			(effects
@@
 			)
 		)
-		(property "Value" "100K 1%"
+		(property "Value" "100k"
 			(at 83.82 173.99 0)
 			(effects
@@
 			)
 		)
-		(property "Datasheet" "https://fscdn.rohm.com/en/products/databook/datasheet/passive/resistor/chip_resistor/mcr-e.pdf"
+		(property "Datasheet" ""
 			(at 82.55 173.99 0)
 			(effects
@@
 		)
 		(property "Description" ""
-			(at 82.55 173.99 0)
-			(effects
-				(font
-					(size 1.27 1.27)
-				)
-				(hide yes)
-			)
-		)
-		(property "Field4" "Farnell"
-			(at 82.55 173.99 0)
-			(effects
-				(font
-					(size 1.27 1.27)
-				)
-				(hide yes)
-			)
-		)
-		(property "Field5" ""
-			(at 82.55 173.99 0)
-			(effects
-				(font
-					(size 1.27 1.27)
-				)
-				(hide yes)
-			)
-		)
-		(property "Field6" "MCR01MZPF1003"
-			(at 82.55 173.99 0)
-			(effects
-				(font
-					(size 1.27 1.27)
-				)
-				(hide yes)
-			)
-		)
-		(property "Field7" "Rohm"
-			(at 82.55 173.99 0)
-			(effects
-				(font
-					(size 1.27 1.27)
-				)
-				(hide yes)
-			)
-		)
-		(property "Part Description" "Resistor 100K M1005 1% 63mW"
-			(at 82.55 173.99 0)
-			(effects
-				(font
-					(size 1.27 1.27)
-				)
-				(hide yes)
-			)
-		)
-		(property "Field8" ""
 			(at 82.55 173.99 0)
 			(effects
@@
 			)
 		)
-		(property "Footprint" ""
+		(property "Footprint" "MountingHole:MountingHole_3.78mm_M2_Pad_TopOnly"
 			(at 251.46 87.63 0)
 			(effects
@@
 			)
 		)
-		(property "Datasheet" "https://fscdn.rohm.com/en/products/databook/datasheet/passive/resistor/chip_resistor/mcr-e.pdf"
+		(property "Datasheet" ""
 			(at 195.58 82.55 0)
 			(effects
@@
 			)
 		)
-		(property "Value" "2.2K 1%"
+		(property "Value" "2k2"
 			(at 114.808 181.483 0)
 			(effects
@@
 			)
 		)
-		(property "Datasheet" "https://fscdn.rohm.com/en/products/databook/datasheet/passive/resistor/chip_resistor/mcr-e.pdf"
+		(property "Datasheet" ""
 			(at 113.03 180.34 0)
 			(effects
@@
 		)
 		(property "Description" ""
-			(at 113.03 180.34 0)
-			(effects
-				(font
-					(size 1.27 1.27)
-				)
-				(hide yes)
-			)
-		)
-		(property "Field4" "Farnell"
-			(at 113.03 180.34 0)
-			(effects
-				(font
-					(size 1.27 1.27)
-				)
-				(hide yes)
-			)
-		)
-		(property "Field6" ""
-			(at 113.03 180.34 0)
-			(effects
-				(font
-					(size 1.27 1.27)
-				)
-				(hide yes)
-			)
-		)
-		(property "Field7" ""
-			(at 113.03 180.34 0)
-			(effects
-				(font
-					(size 1.27 1.27)
-				)
-				(hide yes)
-			)
-		)
-		(property "Part Description" "Resistor 2.2K M1005 1% 63mW"
 			(at 113.03 180.34 0)
 			(effects
@@
 			)
 		)
-		(property "Datasheet" ""
+		(property "Datasheet" "https://www.lcsc.com/product-detail/Cross-slot-countersunk-machine-screw_AOFENG-GB819-M2-0-4X3-304-A2-70-B_C5138758.html"
 			(at 254 142.24 0)
 			(effects
@@
 			)
 		)
-		(property "Description" ""
+		(property "Description" "C5138758"
 			(at 254 142.24 0)
 			(effects
