File: CM5.kicad_sch (KiCad schematic)
At the start: 4 parts, among them J301 Conn_01x03, M303 Compute-Module-4_H1.5mm

Commit message: power symbols
Parts:
- removed J301: Conn_01x03, Connector_PinHeader_2.54mm:PinHeader_1x03_P2.54mm_Vertical, symbol Connector_Generic:Conn_01x03
Connections:
- net PCIE_nRST renamed PCIE_PI.nRST
- no-connect marks 65 -> 67
Other:
- note removed: "Not Fitted header"
Changed lines of the file:
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@@
 	)
 	(junction
+		(at 242.57 57.15)
+		(diameter 0)
+		(color 0 0 0 0)
+	)
+	(junction
 		(at 265.43 149.86)
 		(diameter 1.016)
@@
 	)
 	(no_connect
+		(at 71.12 119.38)
+	)
+	(no_connect
 		(at 345.44 152.4)
 	)
@@
 	)
 	(no_connect
-		(at 161.29 158.75)
-	)
-	(no_connect
 		(at 71.12 124.46)
 	)
@@
 	)
 	(no_connect
+		(at 161.29 124.46)
+	)
+	(no_connect
 		(at 345.44 167.64)
 	)
@@
 	)
 	(no_connect
+		(at 161.29 147.32)
+	)
+	(no_connect
 		(at 71.12 106.68)
 	)
@@
 	)
 	(no_connect
+		(at 71.12 114.3)
+	)
+	(no_connect
 		(at 251.46 162.56)
 	)
@@
 	)
 	(no_connect
-		(at 345.44 91.44)
-	)
-	(no_connect
 		(at 86.36 162.56)
 	)
@@
 	)
 	(bus_entry
+		(at 346.71 91.44)
+		(size 2.54 -2.54)
+		(stroke
+			(width 0)
+			(type default)
+		)
+	)
+	(bus_entry
 		(at 237.49 170.18)
 		(size -2.54 2.54)
@@
 		)
 	)
+	(bus
+		(pts
+			(xy 349.25 57.15) (xy 242.57 57.15)
+		)
+		(stroke
+			(width 0)
+			(type default)
+		)
+	)
 	(wire
 		(pts
@@
 	(wire
 		(pts
-			(xy 69.85 114.3) (xy 86.36 114.3)
+			(xy 71.12 114.3) (xy 86.36 114.3)
 		)
 		(stroke
@@
 	(wire
 		(pts
-			(xy 147.32 124.46) (xy 163.83 124.46)
+			(xy 147.32 124.46) (xy 161.29 124.46)
 		)
 		(stroke
@@
 	(bus
 		(pts
-			(xy 241.3 74.93) (xy 242.57 74.93)
+			(xy 241.3 48.26) (xy 242.57 48.26)
 		)
 		(stroke
@@
 	(bus
 		(pts
-			(xy 345.44 74.93) (xy 345.44 81.28)
+			(xy 345.44 72.39) (xy 345.44 81.28)
 		)
 		(stroke
@@
 		)
 	)
+	(bus
+		(pts
+			(xy 349.25 88.9) (xy 349.25 57.15)
+		)
+		(stroke
+			(width 0)
+			(type default)
+		)
+	)
 	(wire
 		(pts
@@
 	(wire
 		(pts
-			(xy 147.32 147.32) (xy 157.48 147.32)
+			(xy 147.32 147.32) (xy 161.29 147.32)
 		)
 		(stroke
@@
 	(bus
 		(pts
-			(xy 242.57 78.74) (xy 242.57 74.93)
+			(xy 242.57 78.74) (xy 242.57 57.15)
 		)
 		(stroke
@@
 	(wire
 		(pts
-			(xy 69.85 119.38) (xy 86.36 119.38)
+			(xy 71.12 119.38) (xy 86.36 119.38)
 		)
 		(stroke
@@
 		)
 	)
+	(bus
+		(pts
+			(xy 242.57 57.15) (xy 242.57 48.26)
+		)
+		(stroke
+			(width 0)
+			(type default)
+		)
+	)
 	(wire
 		(pts
@@
 	(bus
 		(pts
-			(xy 345.44 74.93) (xy 346.71 74.93)
+			(xy 345.44 72.39) (xy 344.17 72.39)
 		)
 		(stroke
@@
 	(wire
 		(pts
-			(xy 328.93 91.44) (xy 345.44 91.44)
+			(xy 328.93 91.44) (xy 346.71 91.44)
 		)
 		(stroke
@@
 		)
 	)
-	(text "Not Fitted header"
-		(exclude_from_sim no)
-		(at 179.705 180.975 0)
-		(effects
-			(font
-				(size 1.27 1.27)
-			)
-			(justify right bottom)
-		)
-	)
 	(text "CM mechanicals"
 		(exclude_from_sim no)
@@
 		)
 	)
+	(label "GPIO5"
+		(at 71.12 119.38 0)
+		(fields_autoplaced yes)
+		(effects
+			(font
+				(size 1.27 1.27)
+			)
+			(justify left bottom)
+		)
+	)
 	(label "ETH_PI.TRD2_P"
 		(at 177.8 91.44 180)
@@
 		)
 	)
+	(label "GPIO7"
+		(at 161.29 124.46 180)
+		(fields_autoplaced yes)
+		(effects
+			(font
+				(size 1.27 1.27)
+			)
+			(justify right bottom)
+		)
+	)
 	(label "GPIO16"
 		(at 157.48 114.3 180)
@@
 		)
 	)
+	(label "GPIO6"
+		(at 71.12 114.3 0)
+		(fields_autoplaced yes)
+		(effects
+			(font
+				(size 1.27 1.27)
+			)
+			(justify left bottom)
+		)
+	)
 	(label "SYNC_OUT"
 		(at 71.12 99.06 0)
@@
 		)
 	)
-	(label "PCIE_nRST"
+	(label "PCIE_PI.nRST"
 		(at 345.44 91.44 180)
 		(fields_autoplaced yes)
@@
 		)
 	)
-	(hierarchical_label "GPIO7"
-		(shape bidirectional)
-		(at 163.83 124.46 0)
-		(fields_autoplaced yes)
-		(effects
-			(font
-				(size 1.27 1.27)
-			)
-			(justify left)
-		)
-	)
 	(hierarchical_label "DPHY0_P{DPHY}"
 		(shape input)
@@
 	(hierarchical_label "USB_PI{USB}"
 		(shape bidirectional)
-		(at 346.71 74.93 0)
+		(at 344.17 72.39 180)
 		(fields_autoplaced yes)
 		(effects
@@
 				(size 1.27 1.27)
 			)
-			(justify left)
+			(justify right)
 		)
 	)
@@
 		)
 	)
-	(hierarchical_label "GPIO6"
-		(shape bidirectional)
-		(at 69.85 114.3 180)
-		(fields_autoplaced yes)
-		(effects
-			(font
-				(size 1.27 1.27)
-			)
-			(justify right)
-		)
-	)
 	(hierarchical_label "PCIE_PI{PCIE}"
 		(shape input)
-		(at 241.3 74.93 180)
+		(at 241.3 48.26 180)
 		(fields_autoplaced yes)
 		(effects
@@
 	)
 	(hierarchical_label "GPIO_VREF"
-		(shape output)
+		(shape input)
 		(at 69.85 175.26 180)
 		(fields_autoplaced yes)
@@
 		)
 	)
-	(hierarchical_label "GPIO5"
-		(shape bidirectional)
-		(at 69.85 119.38 180)
-		(fields_autoplaced yes)
-		(effects
-			(font
-				(size 1.27 1.27)
-			)
-			(justify right)
-		)
-	)
 	(hierarchical_label "USBOTG_ID"
 		(shape input)
@@
 					(unit 1)
 				)
-			)
-		)
-	)
-	(symbol
-		(lib_id "Connector_Generic:Conn_01x03")
-		(at 170.18 190.5 0)
-		(unit 1)
-		(exclude_from_sim yes)
-		(in_bom no)
-		(on_board no)
-		(dnp yes)
-		(property "Reference" "J301"
-			(at 168.0972 182.4482 0)
-			(effects
-				(font
-					(size 1.27 1.27)
-				)
-			)
-		)
-		(property "Value" "Conn_01x03"
-			(at 168.0972 184.7596 0)
-			(effects
-				(font
-					(size 1.27 1.27)
-				)
-			)
-		)
-		(property "Footprint" "Connector_PinHeader_2.54mm:PinHeader_1x03_P2.54mm_Vertical"
-			(at 170.18 190.5 0)
-			(effects
-				(font
-					(size 1.27 1.27)
-				)
-				(hide yes)
-			)
-		)
-		(property "Datasheet" "~"
-			(at 170.18 190.5 0)
-			(effects
-				(font
-					(size 1.27 1.27)
-				)
-				(hide yes)
-			)
-		)
-		(property "Description" ""
-			(at 170.18 190.5 0)
-			(effects
-				(font
-					(size 1.27 1.27)
-				)
-				(hide yes)
-			)
-		)
-		(property "Field4" "nf"
-			(at 170.18 190.5 0)
-			(effects
-				(font
-					(size 1.27 1.27)
-				)
-				(hide yes)
-			)
-		)
-		(property "Field5" "nf"
-			(at 170.18 190.5 0)
-			(effects
-				(font
-					(size 1.27 1.27)
-				)
-				(hide yes)
-			)
-		)
-		(property "Field6" "nf"
-			(at 170.18 190.5 0)
-			(effects
-				(font
-					(size 1.27 1.27)
-				)
-				(hide yes)
-			)
-		)
-		(property "Field7" "nf"
-			(at 170.18 190.5 0)
-			(effects
-				(font
-					(size 1.27 1.27)
-				)
-				(hide yes)
-			)
-		)
-		(property "Part Description" "3pin 0.1\" connector"
-			(at 170.18 190.5 0)
-			(effects
-				(font
-					(size 1.27 1.27)
-				)
-				(hide yes)
-			)
-		)
-		(pin "1"
-		)
-		(pin "2"
-		)
-		(pin "3"
-		)
-		(instances
-			(project "CM5_CB"
-				(path "/b33e81d6-18a9-4b9d-a239-76a7c253462f/45540f0b-d892-4f71-86ad-b9f245bcefda"
-					(reference "J301")
-					(unit 1)
-				)

Commit message: changed i2c connector and nrpiboot
Connections:
- no-connect marks 67 -> 66
Changed lines of the file:
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@@
 	)
 	(no_connect
-		(at 161.29 195.58)
-	)
-	(no_connect
 		(at 347.98 182.88)
 	)
@@
 	(wire
 		(pts
-			(xy 147.32 195.58) (xy 161.29 195.58)
+			(xy 147.32 195.58) (xy 163.83 195.58)
 		)
 		(stroke
@@
 		)
 	)
-	(label "nRPIBOOT"
-		(at 149.86 195.58 0)
-		(fields_autoplaced yes)
-		(effects
-			(font
-				(size 1.27 1.27)
-			)
-			(justify left bottom)
-		)
-	)
 	(label "HDMI_PI.SCL"
 		(at 240.03 205.74 0)
@@
 		)
 	)
+	(hierarchical_label "nRPIBOOT"
+		(shape input)
+		(at 163.83 195.58 0)
+		(fields_autoplaced yes)
+		(effects
+			(font
+				(size 1.27 1.27)
+			)
+			(justify left)
+		)
+	)
