File: CM5.kicad_sch (KiCad schematic)
At the start: 3 parts, among them M303 Compute-Module-4_H1.5mm

Commit message: swap TX RX M2
Connections:
- no-connect marks 66 -> 64
Changed lines of the file:
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@@
 	)
 	(no_connect
-		(at 71.12 119.38)
-	)
-	(no_connect
 		(at 345.44 152.4)
 	)
@@
 	)
 	(no_connect
-		(at 71.12 144.78)
-	)
-	(no_connect
 		(at 86.36 162.56)
 	)
@@
 	(wire
 		(pts
-			(xy 71.12 144.78) (xy 86.36 144.78)
+			(xy 69.85 144.78) (xy 86.36 144.78)
 		)
 		(stroke
@@
 	(wire
 		(pts
-			(xy 71.12 119.38) (xy 86.36 119.38)
+			(xy 69.85 119.38) (xy 86.36 119.38)
 		)
 		(stroke
@@
 		)
 	)
-	(label "GPIO5"
-		(at 71.12 119.38 0)
-		(fields_autoplaced yes)
-		(effects
-			(font
-				(size 1.27 1.27)
-			)
-			(justify left bottom)
-		)
-	)
 	(label "ETH_PI.TRD2_P"
 		(at 177.8 91.44 180)
@@
 		)
 	)
-	(label "HDMI1_D1_P"
-		(at 251.46 144.78 0)
+	(label "GPIO8"
+		(at 157.48 127 180)
 		(fields_autoplaced yes)
 		(effects
@@
 				(size 1.27 1.27)
 			)
-			(justify left bottom)
+			(justify right bottom)
 		)
 	)
-	(label "GPIO7"
-		(at 161.29 124.46 180)
+	(label "HDMI1_D1_P"
+		(at 251.46 144.78 0)
 		(fields_autoplaced yes)
 		(effects
@@
 				(size 1.27 1.27)
 			)
-			(justify right bottom)
+			(justify left bottom)
 		)
 	)
@@
 		)
 	)
+	(label "GPIO3"
+		(at 71.12 147.32 0)
+		(fields_autoplaced yes)
+		(effects
+			(font
+				(size 1.27 1.27)
+			)
+			(justify left bottom)
+		)
+	)
 	(label "DPHY1_P.D3_P"
 		(at 251.46 200.66 0)
@@
 		)
 	)
+	(label "GPIO2"
+		(at 71.12 149.86 0)
+		(fields_autoplaced yes)
+		(effects
+			(font
+				(size 1.27 1.27)
+			)
+			(justify left bottom)
+		)
+	)
 	(label "HDMI1_SDA"
 		(at 332.74 137.16 0)
@@
 		)
 	)
-	(label "DPHY0_P.D0_P"
-		(at 351.79 101.6 180)
+	(label "GPIO7"
+		(at 157.48 124.46 180)
 		(fields_autoplaced yes)
 		(effects
@@
 		)
 	)
-	(label "HDMI1_SCL"
-		(at 332.74 139.7 0)
+	(label "DPHY0_P.D0_P"
+		(at 351.79 101.6 180)
 		(fields_autoplaced yes)
 		(effects
@@
 				(size 1.27 1.27)
 			)
-			(justify left bottom)
+			(justify right bottom)
 		)
 	)
-	(label "GPIO8"
-		(at 157.48 127 180)
+	(label "HDMI1_SCL"
+		(at 332.74 139.7 0)
 		(fields_autoplaced yes)
 		(effects
@@
 				(size 1.27 1.27)
 			)
-			(justify right bottom)
+			(justify left bottom)
 		)
 	)
@@
 		)
 	)
-	(label "GPIO4"
-		(at 71.12 144.78 0)
-		(fields_autoplaced yes)
-		(effects
-			(font
-				(size 1.27 1.27)
-			)
-			(justify left bottom)
-		)
-	)
 	(label "SD_DAT1"
 		(at 158.75 162.56 180)
@@
 		)
 	)
+	(hierarchical_label "GPIO5"
+		(shape input)
+		(at 69.85 119.38 180)
+		(fields_autoplaced yes)
+		(effects
+			(font
+				(size 1.27 1.27)
+			)
+			(justify right)
+		)
+	)
 	(hierarchical_label "ETH_nLED_ACTIVITY"
 		(shape output)
@@
 		)
 	)
+	(hierarchical_label "GPIO4"
+		(shape input)
+		(at 69.85 144.78 180)
+		(fields_autoplaced yes)
+		(effects
+			(font
+				(size 1.27 1.27)
+			)
+			(justify right)
+		)
+	)
 	(hierarchical_label "GPIO_VREF"
 		(shape input)
@@
 		(fields_autoplaced yes)
 		(effects
-			(font
-				(size 1.27 1.27)
-			)
-			(justify right)
-		)
-	)
-	(hierarchical_label "GPIO3"
-		(shape input)
-		(at 71.12 147.32 180)
-		(fields_autoplaced yes)
-		(effects
-			(font
-				(size 1.27 1.27)
-			)
-			(justify right)
-		)
-	)
-	(hierarchical_label "GPIO2"
-		(shape input)
-		(at 71.12 149.86 180)
-		(fields_autoplaced yes)
-		(effects
