File: HDMI.kicad_sch (KiCad schematic)
At the start: 7 parts, among them J501 690-019-298-412, U405 STMPS2151STR

Commit message: rework for JLC
Parts:
- J501: value 690-019-298-412 -> GT-HD001B-CNNG1; Field4 Farnell -> (none); Field5 2614936 -> (none); Field6 690-019-298-412 -> (none); Field7 EDAC -> (none); Field8 UCON00802 -> (none)
Changed lines of the file:
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@@
 			)
 		)
-		(property "Value" "690-019-298-412"
+		(property "Value" "GT-HD001B-CNNG1"
 			(at 165.1 87.63 0)
 			(effects
@@
 			)
 		)
-		(property "Field4" "Farnell"
+		(property "Field5" ""
 			(at 167.64 55.88 0)
 			(effects
@@
 			)
 		)
-		(property "Field5" "2614936"
-			(at 167.64 55.88 0)
-			(effects
-				(font
-					(size 1.27 1.27)
-				)
-				(hide yes)
-			)
-		)
-		(property "Field6" "690-019-298-412"
-			(at 167.64 55.88 0)
-			(effects
-				(font
-					(size 1.27 1.27)
-				)
-				(hide yes)
-			)
-		)
-		(property "Field7" "EDAC"
+		(property "Field6" ""
 			(at 167.64 55.88 0)
 			(effects
@@
 			(at 167.64 55.88 0)
 			(effects
-				(font
-					(size 1.27 1.27)
-				)
-				(hide yes)
-			)
-		)
-		(property "Field8" "UCON00802"
-			(at 167.64 55.88 0)
-			(effects
