File: CM5_MINIMA_2.kicad_sch (KiCad schematic)
At the start: 16 parts, among them J101 USB_C_Receptacle_USB2.0

Commit message: swap TX RX M2
Parts:
- added R105, R106: 0R, Resistor_SMD:R_0402_1005Metric, symbol Device:R
Connections:
- new net CM5/GPIO4: R106.2
- new net CM5/GPIO5: R105.2
- new net PCIe-M2/RX: R105.1
- new net PCIe-M2/TX: R106.1
Other:
- sheet CM5 ports: added GPIO4, GPIO5; removed GPIO2, GPIO3

Commit message: rework for JLC
Parts:
- removed JP101: nRPIBOOT, Jumper:SolderJumper-2_P1.3mm_Bridged_RoundedPad1.0x1.5mm, symbol Jumper:SolderJumper_2_Bridged
- added SW101: MK-11C04-G013, EasyEDA:SW-SMD_MK-11C04-G013, symbol EasyEDA:MK-11C04-G013
- TP101, TP103: now left out of the parts list
Connections:
- net CM5/nRPIBOOT: now also SW101.C
- net GND: now also SW101.1, SW101.4, SW101.5
- no-connect marks 5 -> 6

Commit message: prod
Parts:
- TP104, TP105, TP106: now left out of the parts list
Changed lines of the file:
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@@
 		(unit 1)
 		(exclude_from_sim no)
-		(in_bom yes)
+		(in_bom no)
 		(on_board yes)
 		(dnp no)
@@
 		(unit 1)
 		(exclude_from_sim no)
-		(in_bom yes)
+		(in_bom no)
 		(on_board yes)
 		(dnp no)
@@
 		(unit 1)
 		(exclude_from_sim no)
-		(in_bom yes)
-		(on_board yes)
-		(dnp no)
+		(in_bom no)
+		(on_board yes)
+		(dnp no)

Commit message: jlc bom polishing
Parts:
- J101: value USB_C_Receptacle_USB2.0 -> TYPEC-305-ACP16H458
- R101: value 2.2K 1% -> 2k2; Field4 Farnell -> (none); Part Description Resistor 2.2K M1005 1% 63mW -> (none)
- R103: value nf -> 0R; Field4 nf -> (none); Field5 nf -> (none); Field6 nf -> (none)
- TP102: now left out of the parts list
Changed lines of the file:
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@@
 			)
 		)
-		(property "Datasheet" "https://fscdn.rohm.com/en/products/databook/datasheet/passive/resistor/chip_resistor/mcr-e.pdf"
+		(property "Datasheet" ""
 			(at 193.04 139.7 0)
 			(effects
@@
 		(unit 1)
 		(exclude_from_sim no)
-		(in_bom yes)
+		(in_bom no)
 		(on_board yes)
 		(dnp no)
@@
 			)
 		)
-		(property "Value" "nf"
+		(property "Value" "0R"
 			(at 196.85 43.18 90)
 			(effects
@@
 			)
 		)
-		(property "Datasheet" "https://fscdn.rohm.com/en/products/databook/datasheet/passive/resistor/chip_resistor/mcr-e.pdf"
+		(property "Datasheet" ""
 			(at 194.31 39.37 0)
 			(effects
@@
 		)
 		(property "Description" ""
-			(at 194.31 39.37 0)
-			(effects
-				(font
-					(size 1.27 1.27)
-				)
-				(hide yes)
-			)
-		)
-		(property "Field4" "nf"
-			(at 194.31 39.37 0)
-			(effects
-				(font
-					(size 1.27 1.27)
-				)
-				(hide yes)
-			)
-		)
-		(property "Field5" "nf"
-			(at 194.31 39.37 0)
-			(effects
-				(font
-					(size 1.27 1.27)
-				)
-				(hide yes)
-			)
-		)
-		(property "Field6" "nf"
 			(at 194.31 39.37 0)
 			(effects
@@
 			)
 		)
-		(property "Value" "USB_C_Receptacle_USB2.0"
+		(property "Value" "TYPEC-305-ACP16H458"
 			(at 35.56 54.61 0)
 			(effects
@@
 			)
 		)
-		(property "Value" "2.2K 1%"
+		(property "Value" "2k2"
 			(at 85.598 51.054 0)
 			(effects
@@
 			)
 		)
-		(property "Datasheet" "https://fscdn.rohm.com/en/products/databook/datasheet/passive/resistor/chip_resistor/mcr-e.pdf"
+		(property "Datasheet" ""
 			(at 95.25 50.8 0)
 			(effects
@@
 			)
 		)
-		(property "Field4" "Farnell"
-			(at 95.25 50.8 0)
-			(effects
-				(font
-					(size 1.27 1.27)
-				)
-				(hide yes)
-			)
-		)
-		(property "Field5" ""
-			(at 95.25 50.8 0)
-			(effects
-				(font
-					(size 1.27 1.27)
-				)
-				(hide yes)
-			)
-		)
 		(property "Field7" ""
 			(at 95.25 50.8 0)
@@
 		)
 		(property "Field6" ""
-			(at 95.25 50.8 0)
-			(effects
-				(font
-					(size 1.27 1.27)
-				)
-				(hide yes)
-			)
-		)
-		(property "Part Description" "Resistor 2.2K M1005 1% 63mW"
 			(at 95.25 50.8 0)
 			(effects
@@
 			)
 		)
-		(property "Datasheet" "https://fscdn.rohm.com/en/products/databook/datasheet/passive/resistor/chip_resistor/mcr-e.pdf"
+		(property "Datasheet" ""
 			(at 193.04 137.16 0)
 			(effects
@@
 			)
 		)
-		(property "Datasheet" "https://fscdn.rohm.com/en/products/databook/datasheet/passive/resistor/chip_resistor/mcr-e.pdf"
+		(property "Datasheet" ""
 			(at 187.96 39.37 0)
 			(effects
