File: IO.kicad_sch (KiCad schematic)
At the start: 17 parts, among them J502 I2C, J503 SPI, J601 JST_SHBM04B-SRSS-TB, SW601 B3U-3000P, SW602 B3U-3000P, U601 SHTC3, U602 SN74LVC1G14DBVR

Commit message: rework for JLC
Parts:
- removed SW602: B3U-3000P, Button_Switch_SMD:SW_SPST_B3U-3000P, symbol Switch:SW_Push
- added SW501: TS-1010A-B, EasyEDA:SW-SMD_TS-1010A-B, symbol EasyEDA:TS-1010A-B
Connections:
- net GND: now also SW501.2, SW501.3, SW501.4, SW501.5
- net PWR_BUT: now also SW501.1
Changed lines of the file:
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@@
+	)
+	(junction
+		(at 31.75 125.73)
+		(diameter 0)
+		(color 0 0 0 0)
 	)
 	(junction
@@
 	)
 	(junction
+		(at 26.67 125.73)
+		(diameter 0)
+		(color 0 0 0 0)
+	)
+	(junction
 		(at 33.02 63.5)
 		(diameter 0)
 		(color 0 0 0 0)
 	)
+	(junction
+		(at 29.21 125.73)
+		(diameter 0)
+		(color 0 0 0 0)
+	)
 	(no_connect
 		(at 171.45 87.63)
@@
 	(wire
 		(pts
-			(xy 33.02 104.14) (xy 33.02 110.49)
-		)
-		(stroke
-			(width 0)
-			(type default)
-		)
-	)
-	(wire
-		(pts
 			(xy 102.87 78.74) (xy 96.52 78.74)
 		)
@@
 	(wire
 		(pts
+			(xy 31.75 125.73) (xy 34.29 125.73)
+		)
+		(stroke
+			(width 0)
+			(type default)
+		)
+	)
+	(wire
+		(pts
 			(xy 66.04 35.56) (xy 68.58 35.56)
 		)
@@
 	(wire
 		(pts
+			(xy 26.67 97.79) (xy 26.67 105.41)
+		)
+		(stroke
+			(width 0)
+			(type default)
+		)
+	)
+	(wire
+		(pts
 			(xy 148.59 74.93) (xy 137.16 74.93)
 		)
@@
 	(wire
 		(pts
+			(xy 29.21 101.6) (xy 34.29 101.6)
+		)
+		(stroke
+			(width 0)
+			(type default)
+		)
+	)
+	(wire
+		(pts
 			(xy 166.37 26.67) (xy 177.8 26.67)
 		)
@@
 	(wire
 		(pts
+			(xy 46.99 118.11) (xy 49.53 118.11)
+		)
+		(stroke
+			(width 0)
+			(type default)
+		)
+	)
+	(wire
+		(pts
 			(xy 148.59 74.93) (xy 151.13 74.93)
 		)
@@
 	(wire
 		(pts
+			(xy 46.99 123.19) (xy 46.99 118.11)
+		)
+		(stroke
+			(width 0)
+			(type default)
+		)
+	)
+	(wire
+		(pts
+			(xy 26.67 125.73) (xy 29.21 125.73)
+		)
+		(stroke
+			(width 0)
+			(type default)
+		)
+	)
+	(wire
+		(pts
 			(xy 33.02 63.5) (xy 33.02 67.31)
 		)
@@
 	(wire
 		(pts
+			(xy 29.21 125.73) (xy 31.75 125.73)
+		)
+		(stroke
+			(width 0)
+			(type default)
+		)
+	)
+	(wire
+		(pts
 			(xy 100.33 88.9) (xy 102.87 88.9)
 		)
@@
 	(wire
 		(pts
-			(xy 45.72 118.11) (xy 49.53 118.11)
-		)
-		(stroke
-			(width 0)
-			(type default)
-		)
-	)
-	(wire
-		(pts
-			(xy 33.02 120.65) (xy 33.02 123.19)
+			(xy 45.72 123.19) (xy 46.99 123.19)
+		)
+		(stroke
+			(width 0)
+			(type default)
+		)
+	)
+	(wire
+		(pts
+			(xy 26.67 125.73) (xy 26.67 128.27)
 		)
 		(stroke
@@
 	(wire
 		(pts
+			(xy 29.21 101.6) (xy 29.21 105.41)
+		)
+		(stroke
+			(width 0)
+			(type default)
+		)
+	)
+	(wire
+		(pts
 			(xy 102.87 71.12) (xy 96.52 71.12)
 		)
@@
 		(pts
 			(xy 102.87 81.28) (xy 96.52 81.28)
+		)
+		(stroke
+			(width 0)
+			(type default)
+		)
+	)
+	(wire
+		(pts
+			(xy 34.29 101.6) (xy 34.29 125.73)
 		)
 		(stroke
@@
 	(hierarchical_label "PWR_BUT"
 		(shape input)
-		(at 33.02 104.14 180)
+		(at 26.67 97.79 180)
 		(fields_autoplaced yes)
 		(effects
@@
 	(hierarchical_label "SDA"
 		(shape bidirectional)
-		(at 45.72 118.11 180)
+		(at 45.72 123.19 180)
 		(fields_autoplaced yes)
 		(effects
@@
 	(symbol
 		(lib_id "power:GND")
-		(at 33.02 123.19 0)
+		(at 26.67 128.27 0)
 		(unit 1)
 		(exclude_from_sim no)
@@
 		(dnp no)
 		(property "Reference" "#PWR0606"
-			(at 33.02 129.54 0)
+			(at 26.67 134.62 0)
 			(effects
 				(font
@@
 		)
 		(property "Value" "GND"
-			(at 33.147 127.5842 0)
+			(at 26.797 132.6642 0)
 			(effects
 				(font
@@
 		)
 		(property "Footprint" ""
-			(at 33.02 123.19 0)
+			(at 26.67 128.27 0)
 			(effects
 				(font
@@
 		)
 		(property "Datasheet" ""
-			(at 33.02 123.19 0)
+			(at 26.67 128.27 0)
 			(effects
 				(font
@@
 		)
 		(property "Description" "Power symbol creates a global label with name \"GND\" , ground"
-			(at 33.02 123.19 0)
+			(at 26.67 128.27 0)
 			(effects
 				(font
@@
 	)
 	(symbol
+		(lib_id "EasyEDA:TS-1010A-B")
+		(at 29.21 115.57 90)
+		(mirror x)
+		(unit 1)
+		(exclude_from_sim no)
+		(in_bom yes)
+		(on_board yes)
+		(dnp no)
+		(property "Reference" "SW501"
+			(at 35.052 99.314 90)
+			(effects
+				(font
+					(size 1.27 1.27)
+				)
+				(justify left)
+			)
+		)
+		(property "Value" "TS-1010A-B"
+			(at 23.114 107.95 0)
+			(effects
+				(font
+					(size 1.27 1.27)
+				)
+				(justify left)
+			)
+		)
+		(property "Footprint" "EasyEDA:SW-SMD_TS-1010A-B"
+			(at 39.37 115.57 0)
+			(effects
+				(font
+					(size 1.27 1.27)
+				)
+				(hide yes)
+			)
+		)
+		(property "Datasheet" "https://lcsc.com/product-detail/Tactile-Switches_XKB-Enterprise-TS-1010A-B_C381059.html"
+			(at 41.91 115.57 0)
+			(effects
+				(font
+					(size 1.27 1.27)
+				)
+				(hide yes)
+			)
+		)
+		(property "Description" ""
+			(at 29.21 115.57 0)
+			(effects
+				(font
+					(size 1.27 1.27)
+				)
+				(hide yes)
+			)
+		)
+		(property "LCSC Part" "C381059"
+			(at 44.45 115.57 0)
+			(effects
+				(font
+					(size 1.27 1.27)
+				)
+				(hide yes)
+			)
+		)
+		(pin "3"
+		)
+		(pin "2"
+		)
+		(pin "1"
+		)
+		(pin "5"
+		)
+		(pin "4"
+		)
+		(instances
+			(project ""
+				(path "/b33e81d6-18a9-4b9d-a239-76a7c253462f/4ce4cfa7-ba20-49b9-8014-333351d4c7f7"
+					(reference "SW501")
+					(unit 1)
+				)
+			)
+		)
+	)
+	(symbol
 		(lib_id "power:+3V3")
 		(at 33.02 48.26 0)
@@
 					(unit 1)
 				)
-			)
-		)
-	)
-	(symbol
-		(lib_id "Switch:SW_Push")
-		(at 33.02 115.57 90)
-		(mirror x)
-		(unit 1)
-		(exclude_from_sim no)
-		(in_bom yes)
-		(on_board yes)
-		(dnp no)
-		(property "Reference" "SW602"
-			(at 18.288 116.84 90)
-			(effects
-				(font
-					(size 1.27 1.27)
-				)
-				(justify right)
-			)
-		)
-		(property "Value" "B3U-3000P"
-			(at 18.288 114.3 90)
-			(effects
-				(font
-					(size 1.27 1.27)
-				)
-				(justify right)
-			)
-		)
-		(property "Footprint" "Button_Switch_SMD:SW_SPST_B3U-3000P"
-			(at 27.94 115.57 0)
-			(effects
-				(font
-					(size 1.27 1.27)
-				)
-				(hide yes)
-			)
-		)
-		(property "Datasheet" "~"
-			(at 27.94 115.57 0)
-			(effects
-				(font
-					(size 1.27 1.27)
-				)
-				(hide yes)
-			)
-		)
-		(property "Description" "Push button switch, generic, two pins"
-			(at 33.02 115.57 0)
-			(effects
-				(font
-					(size 1.27 1.27)
-				)
-				(hide yes)
-			)
-		)
-		(property "P/N" ""
-			(at 30.48 115.57 0)
-			(effects
-				(font
-					(size 1.27 1.27)
-				)
-				(hide yes)
-			)
-		)
-		(pin "1"
-		)
-		(pin "2"
-		)
-		(instances
-			(project "CM5_CB"
-				(path "/b33e81d6-18a9-4b9d-a239-76a7c253462f/4ce4cfa7-ba20-49b9-8014-333351d4c7f7"
-					(reference "SW602")
-					(unit 1)
-				)

Commit message: prod
Parts:
- R501, R502: value 10k -> 2k2
- R605, R606: value 3k3 -> 2k2
Changed lines of the file:
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@@
 			)
 		)
-		(property "Value" "10k"
+		(property "Value" "2k2"
 			(at 151.13 68.58 90)
 			(effects
@@
 			)
 		)
-		(property "Value" "10k"
+		(property "Value" "2k2"
 			(at 158.75 68.58 90)
 			(effects
@@
 		(fields_autoplaced yes)
 		(property "Reference" "R606"
-			(at 140.97 30.48 0)
+			(at 140.97 30.4799 0)
 			(effects
 				(font
@@
 			)
 		)
-		(property "Value" "3k3"
-			(at 140.97 33.02 0)
+		(property "Value" "2k2"
+			(at 140.97 33.0199 0)
 			(effects
 				(font
@@
 		(fields_autoplaced yes)
 		(property "Reference" "R605"
-			(at 91.44 30.48 0)
+			(at 91.44 30.4799 0)
 			(effects
 				(font
@@
 			)
 		)
-		(property "Value" "3k3"
-			(at 91.44 33.02 0)
-			(effects
-				(font
+		(property "Value" "2k2"
+			(at 91.44 33.0199 0)
+			(effects
+				(font

Commit message: jlc bom polishing
Parts:
- R601: dni DNI -> (none)
- SW601: value B3U-3000P -> B3U-3100-P
Changed lines of the file:
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@@
 			)
 		)
-		(property "Datasheet" "~"
+		(property "Datasheet" ""
 			(at 151.13 68.58 0)
 			(effects
@@
 			)
 		)
-		(property "Datasheet" "~"
+		(property "Datasheet" ""
 			(at 158.75 68.58 0)
 			(effects
@@
 			)
 		)
-		(property "dni" "DNI"
-			(at 35.56 58.42 0)
-			(effects
-				(font
-					(size 1.27 1.27)
-				)
-				(justify left)
-			)
-		)
 		(pin "1"
 		)
@@
 			)
 		)
-		(property "Value" "B3U-3000P"
+		(property "Value" "B3U-3100-P"
 			(at 18.288 71.12 90)
 			(effects
