File: USB.kicad_sch (KiCad schematic)
At the start: 9 parts, among them U701 AP22653W6

Commit message: jlc bom polishing
Parts:
- R701: value 15K 1% -> 15k
Changed lines of the file:
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@@
 			)
 		)
-		(property "Value" "15K 1%"
+		(property "Value" "15k"
 			(at 124.46 35.56 90)
 			(effects
@@
 			)
 		)
-		(property "Datasheet" "https://fscdn.rohm.com/en/products/databook/datasheet/passive/resistor/chip_resistor/mcr-e.pdf"
+		(property "Datasheet" ""
 			(at 124.46 39.37 0)
 			(effects
