File: CM5_MINIMA_2.kicad_pcb (KiCad board)
At the start: 6 copper layers, 54.6 x 57.1 mm, 101 parts, among them J101 USB_C_Receptacle_USB2.0, J501 GT-HD001B-CNNG1, J502 I2C, J503 SPI, J601 JST_SHBM04B-SRSS-TB, J701 Bus_M.2_Socket_M, J802 Conn_01x22_Female, SW101 MK-11C04-G013, SW501 TS-1010A-B, T401 7498111120AR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

Commit message: jlc bom polishing
Parts:
- added M701: M.2 Solder Nut, MountingHole:MountingHole_3.78mm_M2_Pad_TopOnly, F.Cu at (113.6, 58.9)
- J101: value USB_C_Receptacle_USB2.0 -> TYPEC-305-ACP16H458
- R101, R706: value 2.2K 1% -> 2k2
- R103: value nf -> 0R
- R701: value 15K 1% -> 15k
- R704: value 100K 1% -> 100k
- R705: value 10K 1% -> 10k
